File: Electrónica/Player_v0.3_simplified.brd (EAGLE design)
At the start: 104.9 x 75.1 mm, 61 parts, among them IC1 7805DT, IC2 7805DT, IC3 7805DT, IC4 7805DT

Commit message: - unified Peripherals and boards
Parts:
- removed C5, C6, C7, C8: (no value), rcl:E2,5-5
- removed IC3, IC4: 7805DT, linear:TO252
- removed LED10, LED11, LED12, LED7, LED8, LED9: (no value), adafruit:LED5MM
- removed S10, S11, S12, S13, S14, S8, S9: SWITCH-MOMENTARY-2PTH, SparkFun-Electromechanical:TACTILE-PTH
- removed SG2: F/DB18, buzzer:F/DB18
- removed VIN2, VIN3, X1, X2, X29, X30, X33, X34, X35, X36, X37, X38, X39, X40, X41, X42: (no value), con-molex:KK-156-2
- added LED1, LED2, LED3, LED4, LED5, LED6: (no value), adafruit:LED5MM
- added S1, S2, S3, S4, S5, S6, S7: SWITCH-MOMENTARY-2PTH, SparkFun-Electromechanical:TACTILE-PTH
- added SG1: F/DB18, buzzer:F/DB18
- added X11, X12, X13, X14, X15, X16, X24, X25, X26, X27, X28, X3, X31, X32: (no value), con-molex:KK-156-2
Connections:
- removed net N$22: S8.3, X1.1
- removed net N$33: S9.3, X33.1
- removed net N$54: S10.3, X34.1
- removed net N$56: S11.3, X35.1
- removed net N$58: S12.3, X36.1
- removed net N$60: S13.3, X37.1
- removed net N$62: LED7.A, X29.1
- removed net N$64: S14.3, X2.1
- removed net N$66: S14.1, X2.2
- removed net N$67: S13.1, X37.2
- removed net N$68: S12.1, X36.2
- removed net N$69: S11.1, X35.2
- removed net N$70: S10.1, X34.2
- removed net N$71: S9.1, X33.2
- removed net N$72: S8.1, X1.2
- removed net N$80: LED7.K, X29.2
- removed net N$81: LED8.A, X38.1
- removed net N$82: LED8.K, X38.2
- removed net N$83: LED9.A, X39.1
- removed net N$84: LED9.K, X39.2
- removed net N$85: LED10.A, X40.1
- removed net N$86: LED10.K, X40.2
- removed net N$87: LED11.A, X41.1
- removed net N$88: LED11.K, X41.2
- removed net N$89: LED12.A, X42.1
- removed net N$90: LED12.K, X42.2
- removed net N$91: SG2.+, X30.1
- removed net N$92: SG2.-, X30.2
- removed net VCC: C5.+, C7.+, IC3.2, IC4.2
- new net N$16: LED1.A, X3.1
- new net N$25: LED1.K, X3.2
- new net N$26: LED2.A, X12.1
- new net N$27: LED2.K, X12.2
- new net N$29: LED3.A, X13.1
- new net N$30: LED3.K, X13.2
- new net N$31: LED4.A, X14.1
- new net N$34: LED4.K, X14.2
- new net N$35: LED5.A, X15.1
- new net N$36: LED5.K, X15.2
- new net N$37: LED6.A, X16.1
- new net N$38: LED6.K, X16.2
- new net N$47: SG1.+, X11.1
- new net N$48: SG1.-, X11.2
- new net N$49: S1.3, X24.1
- new net N$50: S2.3, X26.1
- new net N$51: S3.3, X27.1
- new net N$52: S4.3, X28.1
- new net N$53: S5.3, X31.1
- new net N$55: S6.3, X32.1
- new net N$57: S7.3, X25.1
- new net N$59: S7.1, X25.2
- new net N$61: S6.1, X32.2
- new net N$63: S5.1, X31.2
- new net N$65: S4.1, X28.2
- new net N$73: S3.1, X27.2
- new net N$74: S2.1, X26.2
- new net N$75: S1.1, X24.2
- net +12V: no longer C6.+, C8.+, IC3.1, IC4.1, VIN2.2, VIN3.2
- net GND: no longer C5.-, C6.-, C7.-, C8.-, VIN2.1, VIN3.1
